Commit message: added laser in gazebo

File: taurob_mi_description/urdf/inertia_tensors.urdf.xacro (robot description, xacro)
@@ -1,4 +1,3 @@
-<?xml version="1.0"?>
-<robot xmlns:xacro="http://ros.org/wiki/xacro">
+<robot xmlns:xacro="http://www.ros.org/wiki/xacro" name="taurob_mi">
   <xacro:macro name="inertial_cuboid" params="mass x_length y_length z_length">
     <inertial>

File: taurob_mi_description/urdf/taurob_mi.urdf.xacro (robot description, xacro)
@@ -1,3 +1,2 @@
-<?xml version="1.0"?>
 <robot xmlns:xacro="http://www.ros.org/wiki/xacro" name="taurob_mi">
   <xacro:property name="flipper_offset_x" value="0.205"/>
@@ -8,3 +7,5 @@
   <xacro:include filename="$(find taurob_mi_description)/urdf/taurob_mi_chassis.urdf.xacro"/>
   <tracker_chassis_macro/>
+   <!--LASER-->
+   <xacro:include filename="$(find taurob_mi_description)/urdf/hokuyo_utm30lx.urdf.xacro" />
 </robot>

File: taurob_mi_description/urdf/taurob_mi_chassis.urdf.xacro (robot description, xacro)
@@ -1,3 +1,2 @@
-<?xml version="1.0"?>
 <robot xmlns:xacro="http://www.ros.org/wiki/xacro" name="taurob_mi">
   <xacro:include filename="$(find taurob_mi_description)/urdf/inertia_tensors.urdf.xacro"/>
@@ -44,5 +43,5 @@
         <origin xyz="0.0 0.0 0.0" rpy="0 0 0"/>
         <geometry>
-          <mesh filename="package://taurob_mi_description/meshes/tracker_chassis.dae"/>
+          <mesh filename="package://taurob_mi_description/meshes/taurob/tracker_chassis.dae"/>
         </geometry>
       </visual>
@@ -67,3 +66,16 @@
     </link>
   </xacro:macro>
+<!-- gazebo plugins to control and simulate robot -->
+ <gazebo>
+    <plugin name="p3d_base_controller" filename="libgazebo_ros_p3d.so">
+      <alwaysOn>true</alwaysOn>
+      <updateRate>50.0</updateRate>
+      <bodyName>base_link</bodyName>
+      <topicName>ground_truth/state</topicName>
+      <gaussianNoise>0.01</gaussianNoise>
+      <frameName>world</frameName>
+      <xyzOffsets>0 0 0</xyzOffsets>
+      <rpyOffsets>0 0 0</rpyOffsets>
+    </plugin>
+  </gazebo>
 </robot>

File: taurob_mi_description/urdf/tracker_standalone.urdf.xacro (robot description, xacro)
@@ -1,5 +1,5 @@
 <?xml version="1.0"?>
 <robot name="taurob_tracker"
-    xmlns:xacro="http://playerstage.sourceforge.net/gazebo/xmlschema/#interface">
+    xmlns:xacro="http://ros.org/wiki/xacro">
     <property name="flipper_offset_x" value="0.205" />
     <property name="flipper_offset_y" value="0.15" />
@@ -20,4 +20,4 @@
       <origin xyz="0.0 0 0.0" rpy="0 ${45 * M_PI/180.0} 0"/>
     </spinning_hokuyo_utm30lx_lidar_mount_offset_macro >
-    -->
+ -->
 </robot>
