Commit message: updated and unified model with laser and schunk arm

File: taurob_mi_description/urdf/hokuyo_utm30lx.urdf.xacro (robot description, xacro)
@@ -1,6 +1,6 @@
-<robot xmlns:xacro="http://ros.org/wiki/xacro">
+<robot xmlns:xacro="http://www.ros.org/wiki/xacro">
     <xacro:property name="M_PI" value="3.1415926535897931" />
       <joint name="hokuyo_joint" type="fixed">
-        <origin xyz="0.15 0 0.1" rpy="0 0 0"/>
+        <origin xyz="0.2 0 0.1" rpy="0 0 0"/>
         <parent link="chassis_link"/>
         <child link="hokuyo_link"/>

File: taurob_mi_description/urdf/taurob_mi.urdf.xacro (robot description, xacro)
@@ -5,10 +5,15 @@
   <xacro:property name="M_PI" value="3.14159"/>
   <xacro:property name="angle_deg" value="45"/>
+  <!-- common stuff -->
+  <xacro:include filename="$(find taurob_schunk_lwa4d)/urdf/common.xacro" />
+  <xacro:include filename="$(find taurob_schunk_lwa4d)/urdf/materials.urdf.xacro" />
  <!--main chassis-->
   <xacro:include filename="$(find taurob_mi_description)/urdf/taurob_mi_chassis.urdf.xacro"/>
- <!--schunk lwa4d arm-->
-  <xacro:include filename="$(find taurob_schunk_lwa4d)/urdf/taurob_schunk_lwa4d.urdf.xacro"/>
-  <tracker_chassis_macro/>
  <!--LASER-->
   <xacro:include filename="$(find taurob_mi_description)/urdf/hokuyo_utm30lx.urdf.xacro" />
+<!--schunk lwa4d arm-->
+  <xacro:include filename="$(find taurob_schunk_lwa4d)/urdf/lwa4d/lwa4d.urdf.xacro" />
+  <xacro:schunk_lwa4d name="arm" parent="base_link" has_podest="false">
+    <origin xyz="0.12 0 0.185" rpy="0 0 ${M_PI/2}"/>
+  </xacro:schunk_lwa4d>
 </robot>

File: taurob_mi_description/urdf/taurob_mi_chassis.gazebo.xacro (robot description, xacro)
@@ -1,22 +1,17 @@
-<?xml version="1.0"?>
-<!--
-Two options available:
-* tracker_chassis_gazebo_force_based_move_macro: Simulates tracks by directly applying force to base_link
-* tracker_chassis_gazebo_fake_wheels_macro: Simulates tracks via multiple wheels attached to robot
-See https://bitbucket.org/osrf/gazebo/issues/863/tracksdriveplugin for some further info
--->
-<robot name="taurob_tracker"
-       xmlns:xacro="http://playerstage.sourceforge.net/gazebo/xmlschema/#interface"
-       xmlns:controller="http://playerstage.sourceforge.net/gazebo/xmlschema/#controller"
-       xmlns:interface="http://playerstage.sourceforge.net/gazebo/xmlschema/#interface">
-  <xacro:include filename="$(find taurob_mi_description)/urdf/inertia_tensors.urdf.xacro" />
-  <!--  <xacro:include filename="$(find taurob_mi_description)/urdf/tracked_wheel.urdf.xacro" />-->
-  <property name="wheel_radius_big" value="0.085" />
-  <property name="wheel_length" value="0.02" />
-  <property name="wheel_size_y" value="0.02" />
-  <property name="wheel_offset_y" value="0.25" />
-  <property name="wheel_offset_z_from_base_link" value="-0.0" />
-  <xacro:property name="wheel_radius" value="0.2" />
-  <xacro:property name="diff_z_offset" value="-0.12" />
+<robot xmlns:xacro="http://www.ros.org/wiki/xacro">
+<!-- pose 3d plugin for ground truth of taurob -->
+  <gazebo>
+    <plugin name="p3d_base_controller" filename="libgazebo_ros_p3d.so">
+      <alwaysOn>true</alwaysOn>
+      <updateRate>50.0</updateRate>
+      <bodyName>base_link</bodyName>
+      <topicName>taurob/pose_ground_truth</topicName>
+      <gaussianNoise>0.01</gaussianNoise>
+      <frameName>map</frameName>
+      <xyzOffsets>0 0 0</xyzOffsets>
+      <rpyOffsets>0 0 0</rpyOffsets>
+    </plugin>
+  </gazebo>
+<!-- imu for taurob -->
   <gazebo>
     <plugin name="imu_controller" filename="libhector_gazebo_ros_imu.so">
@@ -24,5 +19,5 @@
       <updateRate>50.0</updateRate>
       <bodyName>base_link</bodyName>
-      <topicName>/imu/data</topicName>
+      <topicName>taurob/imu/data</topicName>
       <accelDrift>0.0 0.0 0.0</accelDrift>
       <accelGaussianNoise>0.1 0.1 0.1</accelGaussianNoise>
@@ -32,128 +27,9 @@
       <headingGaussianNoise>0.05</headingGaussianNoise>
     </plugin>
-    <plugin name="p3d_base_controller" filename="libgazebo_ros_p3d.so">
-      <alwaysOn>true</alwaysOn>
-      <updateRate>50.0</updateRate>
-      <bodyName>base_link</bodyName>
-      <topicName>ground_truth/state</topicName>
-      <gaussianNoise>0.01</gaussianNoise>
-      <frameName>world</frameName>
-      <xyzOffsets>0 0 0</xyzOffsets>
-      <rpyOffsets>0 0 0</rpyOffsets>
-    </plugin>
-    <!-- ros_control plugin -->
+  </gazebo>
+<!-- ros_control plugin
     <plugin name="gazebo_ros_control" filename="libgazebo_ros_control.so">
       <robotNamespace>tracker_controllers</robotNamespace>
     </plugin>
-    <!-- ros_control plugin -->
-    <plugin name="gazebo_ros_control_select_joints" filename="libgazebo_ros_control_select_joints.so">
-      <robotNamespace>flipper_control</robotNamespace>
-      <joints>flipper_joint_1</joints>
-    </plugin>
-  </gazebo>
-  <macro name="tracker_flipper_move_gazebo_macro">
-      <gazebo>
-        <plugin name="mimic_flipper_joint_0" filename="libroboticsgroup_gazebo_mimic_joint_plugin.so">
-            <joint>flipper_joint_1</joint>
-            <mimicJoint>flipper_joint_0</mimicJoint>
-            <multiplier>0.46</multiplier>
-            <offset>0.0</offset>
-            <maxEffort>10000</maxEffort>
-            <hasPID/>
-        </plugin>
-    </gazebo>
-  </macro>
-  <macro name="tracker_chassis_gazebo_force_based_move_macro">
-    <gazebo reference="chassis_link">
-      <mu1>0.0</mu1>
-      <mu2>0.0</mu2>
-      <kp>1000000.0</kp>
-      <kd>100.0</kd>
-      <minDepth>0.001</minDepth>
-      <maxVel>1.0</maxVel>
-      <!--<material>Gazebo/Grey</material>-->
-    </gazebo>
-    <gazebo reference="base_link">
-      <mu1>0.0</mu1>
-      <mu2>0.0</mu2>
-      <kp>1000000.0</kp>
-      <kd>100.0</kd>
-      <minDepth>0.001</minDepth>
-      <maxVel>1.0</maxVel>
-    </gazebo>
-    <gazebo reference="flipper_link_0">
-      <mu1>200.0</mu1>
-      <mu2>100.0</mu2>
-      <kp>500.0</kp>
-      <kd>100.0</kd>
-      <minDepth>0.001</minDepth>
-      <maxVel>1.0</maxVel>
-      <material>Gazebo/Black</material>
-    </gazebo>
-    <gazebo reference="flipper_link_1">
-      <mu1>0.0</mu1>
-      <mu2>0.0</mu2>
-      <kp>1000000.0</kp>
-      <kd>100.0</kd>
-      <minDepth>0.001</minDepth>
-      <maxVel>1.0</maxVel>
-      <material>Gazebo/Black</material>
-    </gazebo>
-    <gazebo>
-      <plugin name="force_based_move_controller" filename="libgazebo_ros_force_based_move.so">
-        <commandTopic>/cmd_vel_raw</commandTopic>
-        <odometryTopic>odom</odometryTopic>
-        <odometryFrame>odom</odometryFrame>
-        <odometryRate>20.0</odometryRate>
-        <robotBaseFrame>base_link</robotBaseFrame>
-        <yaw_velocity_p_gain>250</yaw_velocity_p_gain>
-        <publishOdometryTf>1</publishOdometryTf>
-      </plugin>
-    </gazebo>
-  </macro>
-  <macro name="tracker_chassis_gazebo_fake_wheels_macro">
-    <!--<tracked_wheel parent="base_link" prefix="left_0" offset_x= "0.21100" offset_y = "${wheel_offset_y}" offset_z = "${wheel_offset_z_from_base_link}" reflect="1" wheel_radius="${wheel_radius_big}"/>-->
-    <tracked_wheel parent="base_link" prefix="left_1" offset_x= "-0.1" offset_y = "${wheel_offset_y}" offset_z = "${wheel_offset_z_from_base_link}" reflect="1" wheel_radius="${wheel_radius_big}"/>
-    <!--<tracked_wheel parent="base_link" prefix="left_2" offset_x= "-0.21100" offset_y = "${wheel_offset_y}" offset_z = "${wheel_offset_z_from_base_link}" reflect="1" wheel_radius="${wheel_radius_big}"/>-->
-    <tracked_wheel parent="base_link" prefix="left_3" offset_x= "0.10" offset_y = "${wheel_offset_y}" offset_z = "${wheel_offset_z_from_base_link}" reflect="1" wheel_radius="${wheel_radius_big}"/>
-    <!--<tracked_wheel parent="base_link" prefix="left_4" offset_x= "-0.10550" offset_y = "${wheel_offset_y}" offset_z = "${wheel_offset_z_from_base_link}" reflect="1" wheel_radius="${wheel_radius_big}"/>-->
-    <!--<tracked_wheel parent="base_link" prefix="right_0" offset_x= "0.21100" offset_y = "-${wheel_offset_y}" offset_z = "${wheel_offset_z_from_base_link}" reflect="1" wheel_radius="${wheel_radius_big}"/>-->
-    <tracked_wheel parent="base_link" prefix="right_1" offset_x= "-0.1" offset_y = "-${wheel_offset_y}" offset_z = "${wheel_offset_z_from_base_link}" reflect="1" wheel_radius="${wheel_radius_big}"/>
-    <!--<tracked_wheel parent="base_link" prefix="right_2" offset_x= "-0.21100" offset_y = "-${wheel_offset_y}" offset_z = "${wheel_offset_z_from_base_link}" reflect="1" wheel_radius="${wheel_radius_big}"/>-->
-    <tracked_wheel parent="base_link" prefix="right_3" offset_x= "0.1" offset_y = "-${wheel_offset_y}" offset_z = "${wheel_offset_z_from_base_link}" reflect="1" wheel_radius="${wheel_radius_big}"/>
-    <!--<tracked_wheel parent="base_link" prefix="right_4" offset_x= "0.10550" offset_y = "-${wheel_offset_y}" offset_z = "${wheel_offset_z_from_base_link}" reflect="1" wheel_radius="${wheel_radius_big}"/>-->
-    <gazebo reference="flipper_link">
-      <mu1>0.0</mu1>
-      <mu2>0.0</mu2>
-      <kp>1000000.0</kp>
-      <kd>100.0</kd>
-      <minDepth>0.001</minDepth>
-      <maxVel>1.0</maxVel>
-    </gazebo>
-    <gazebo reference="base_link">
-      <mu1>0.0</mu1>
-      <mu2>0.0</mu2>
-      <kp>1000000.0</kp>
-      <kd>100.0</kd>
-      <minDepth>0.001</minDepth>
-      <maxVel>1.0</maxVel>
-    </gazebo>
-    <gazebo>
-      <plugin name="diffdrive_plugin_multiwheel" filename="libdiffdrive_plugin_multi_wheel.so">
-        <alwaysOn>true</alwaysOn>
-        <updateRate>25.0</updateRate>
-        <leftJoints>left_1_wheel_joint  left_3_wheel_joint </leftJoints>
-        <rightJoints>right_1_wheel_joint right_3_wheel_joint</rightJoints>
-        <wheelSeparation>${wheel_offset_y*2}</wheelSeparation>
-        <wheelDiameter>${wheel_radius_big*2}</wheelDiameter>
-        <torque>50000</torque>
-        <interface:position name="position_iface_2"/>
-        <robotNamespace>/</robotNamespace>
-        <robotBaseFrame>base_link</robotBaseFrame>
-        <commandTopic>/cmd_vel_raw</commandTopic>
-        <publishOdometryTf>0</publishOdometryTf>
-        <publishOdometryMsg>1</publishOdometryMsg>
-      </plugin>
-    </gazebo>
-  </macro>
+-->
 </robot>

File: taurob_mi_description/urdf/taurob_mi_chassis.urdf.xacro (robot description, xacro)
@@ -1,4 +1,5 @@
-<robot xmlns:xacro="http://www.ros.org/wiki/xacro" name="taurob_mi">
+<robot xmlns:xacro="http://www.ros.org/wiki/xacro">
   <xacro:include filename="$(find taurob_mi_description)/urdf/inertia_tensors.urdf.xacro"/>
+  <xacro:include filename="$(find taurob_mi_description)/urdf/taurob_mi_chassis.gazebo.xacro" />
   <xacro:property name="base_size_x" value="${0.365*2}"/>
   <xacro:property name="base_size_y" value="0.24"/>
@@ -6,5 +7,4 @@
   <xacro:property name="base_offset_x" value="-0.122"/>
   <xacro:property name="base_offset_z" value="-0.05"/>
-  <xacro:macro name="tracker_chassis_macro">
     <link name="base_link"/>
     <joint name="chassis_joint" type="fixed">
@@ -65,44 +65,3 @@
       </collision>
     </link>
-  </xacro:macro>
-<!-- gazebo ROS plugins -->
- <gazebo>
-    <plugin name="p3d_base_controller" filename="libgazebo_ros_p3d.so">
-      <alwaysOn>true</alwaysOn>
-      <updateRate>50.0</updateRate>
-      <bodyName>base_link</bodyName>
-      <topicName>ground_truth/state</topicName>
-      <gaussianNoise>0.01</gaussianNoise>
-      <frameName>world</frameName>
-      <xyzOffsets>0 0 0</xyzOffsets>
-      <rpyOffsets>0 0 0</rpyOffsets>
-    </plugin>
-    <plugin name="imu_controller" filename="libhector_gazebo_ros_imu.so">
-      <alwaysOn>true</alwaysOn>
-      <updateRate>50.0</updateRate>
-      <bodyName>base_link</bodyName>
-      <topicName>/imu/data</topicName>
-      <accelDrift>0.0 0.0 0.0</accelDrift>
-      <accelGaussianNoise>0.1 0.1 0.1</accelGaussianNoise>
-      <rateDrift>0.0 0.0 0.0</rateDrift>
-      <rateGaussianNoise>0.05 0.05 0.05</rateGaussianNoise>
-      <headingDrift>0.0</headingDrift>
-      <headingGaussianNoise>0.05</headingGaussianNoise>
-    </plugin>
-<!-- We need to model the wheel joints for that and take some values from hector e.g. torque -->
-  <plugin name="skid_steer_drive_controller" filename="libgazebo_ros_skid_steer_drive.so">
-    <updateRate>100.0</updateRate>
-    <robotNamespace>/</robotNamespace>
-    <leftFrontJoint>front_left_wheel_joint</leftFrontJoint>
-    <rightFrontJoint>front_right_wheel_joint</rightFrontJoint>
-    <leftRearJoint>back_left_wheel_joint</leftRearJoint>
-    <rightRearJoint>back_right_wheel_joint</rightRearJoint>
-    <wheelSeparation>0.4</wheelSeparation>
-    <wheelDiameter>0.215</wheelDiameter>
-    <robotBaseFrame>base_link</robotBaseFrame>
-    <torque>50000</torque>
-    <topicName>cmd_vel</topicName>
-    <broadcastTF>true</broadcastTF>
-  </plugin>
-  </gazebo>
 </robot>
