Commit message: unified model taurob + arm

File: taurob_erl_description/urdf/hokuyo_utm30lx.urdf.xacro (robot description, xacro)
@@ -1,6 +1,7 @@
+<?xml version="1.0"?>
 <robot xmlns:xacro="http://www.ros.org/wiki/xacro">
     <xacro:property name="M_PI" value="3.1415926535897931" />
       <joint name="hokuyo_joint" type="fixed">
-        <origin xyz="0.2 0 0.1" rpy="0 0 0"/>
+        <origin xyz="0.2 0 0.07" rpy="0 0 0"/>
         <parent link="chassis_link"/>
         <child link="hokuyo_link"/>

File: taurob_erl_description/urdf/taurob_erl.urdf.xacro (robot description, xacro)
@@ -1,13 +1,17 @@
 <?xml version="1.0"?>
-<robot name="taurob_tracker" xmlns:xacro="http://www.ros.org/wiki/xacro">
+<robot name="taurob_erl" xmlns:xacro="http://www.ros.org/wiki/xacro">
   <!--Required to quickly work around bug in collada_urdf (https://github.com/ros/robot_model/issues/132)-->
   <xacro:property name="box_scale_factor" value="1.0" />
   <xacro:property name="M_PI" value="3.14159"/>
   <xacro:include filename="$(find taurob_erl_description)/urdf/taurob_chassis.urdf.xacro.xml" />
-  <xacro:tracker_chassis_macro />
   <xacro:include filename="$(find taurob_erl_description)/urdf/taurob_chassis_cameras.urdf.xacro.xml" />
   <xacro:tracker_chassis_cameras_macro />
   <!--LASER-->
    <xacro:include filename="$(find taurob_erl_description)/urdf/hokuyo_utm30lx.urdf.xacro" />
+  <!--schunk lwa4d arm-->
+    <xacro:include filename="$(find taurob_schunk_lwa4d)/urdf/lwa4d/lwa4d.urdf.xacro" />
+    <xacro:schunk_lwa4d name="arm" parent="base_link" has_podest="true" use_factory_settings="true">
+      <origin xyz="0.12 0 0.185" rpy="0 0 ${M_PI/2}" />
+    </xacro:schunk_lwa4d>
   <!--
   <xacro:generic_camera name="left" parent="base_link" ros_topic="image_mono" cam_info_topic="camera_info" update_rate="10" res_x="640" res_y="480" image_format="L8" hfov="120">

Commit message: updated and fixed unified model

File: taurob_erl_description/urdf/hokuyo_utm30lx.urdf.xacro (robot description, xacro)
@@ -3,5 +3,5 @@
     <xacro:property name="M_PI" value="3.1415926535897931" />
       <joint name="hokuyo_joint" type="fixed">
-        <origin xyz="0.2 0 0.07" rpy="0 0 0"/>
+        <origin xyz="0.17 0 0.05" rpy="0 0 0"/>
         <parent link="chassis_link"/>
         <child link="hokuyo_link"/>

File: taurob_erl_description/urdf/taurob_erl.urdf.xacro (robot description, xacro)
@@ -12,5 +12,5 @@
     <xacro:include filename="$(find taurob_schunk_lwa4d)/urdf/lwa4d/lwa4d.urdf.xacro" />
     <xacro:schunk_lwa4d name="arm" parent="base_link" has_podest="true" use_factory_settings="true">
-      <origin xyz="0.12 0 0.185" rpy="0 0 ${M_PI/2}" />
+      <origin xyz="0.12 0 0.185" rpy="0 0 0" />
     </xacro:schunk_lwa4d>
   <!--

Commit message: several fixes + gripper unified model added

File: taurob_erl_description/urdf/hokuyo_utm30lx.urdf.xacro (robot description, xacro)
@@ -17,5 +17,5 @@
           <origin xyz="0 0 0" rpy="0 0 0" />
           <geometry>
-          <mesh filename="package://taurob_mi_description/meshes/hokuyo_utm30lx/hokuyo_utm_30lx.dae"/>
+          <mesh filename="package://taurob_erl_description/meshes/hokuyo_utm30lx/hokuyo_utm_30lx.dae"/>
           </geometry>
          </visual>
@@ -24,5 +24,5 @@
           <geometry>
           <box size="0.058 0.058 0.087" />
-          <!--<mesh filename="package://taurob_mi_description/meshes/hokuyo_utm30lx/hokuyo_utm_30lx.stl"/>-->
+          <!--<mesh filename="package://taurob_erl_description/meshes/hokuyo_utm30lx/hokuyo_utm_30lx.stl"/>-->
           </geometry>
         </collision>

File: taurob_erl_description/urdf/taurob_erl.urdf.xacro (robot description, xacro)
@@ -14,4 +14,9 @@
       <origin xyz="0.12 0 0.185" rpy="0 0 0" />
     </xacro:schunk_lwa4d>
+    <!-- schunk pg70 -->
+    <xacro:include filename="$(find erl_schunk_pg70)/urdf/pg70/pg70.urdf.xacro" />
+    <xacro:schunk_pg70 name="pg70" parent="arm_ee_link">
+      <origin xyz="0 0 0" rpy="0 0 0" />
+    </xacro:schunk_pg70>
   <!--
   <xacro:generic_camera name="left" parent="base_link" ros_topic="image_mono" cam_info_topic="camera_info" update_rate="10" res_x="640" res_y="480" image_format="L8" hfov="120">

Commit message: problem with laser model fixed

File: taurob_erl_description/urdf/hokuyo_utm30lx.urdf.xacro (robot description, xacro)
@@ -17,5 +17,5 @@
           <origin xyz="0 0 0" rpy="0 0 0" />
           <geometry>
-          <mesh filename="package://taurob_erl_description/meshes/hokuyo_utm30lx/hokuyo_utm_30lx.dae"/>
+          <mesh filename="package://taurob_erl_description/meshes/hokuyo_utm_30lx.dae"/>
           </geometry>
          </visual>
@@ -24,5 +24,5 @@
           <geometry>
           <box size="0.058 0.058 0.087" />
-          <!--<mesh filename="package://taurob_erl_description/meshes/hokuyo_utm30lx/hokuyo_utm_30lx.stl"/>-->
+          <!--<mesh filename="package://taurob_erl_description/meshes/hokuyo_utm_30lx.stl"/>-->
           </geometry>
         </collision>

File: taurob_erl_description/urdf/taurob_erl.urdf.xacro (robot description, xacro)
@@ -5,8 +5,10 @@
   <xacro:property name="M_PI" value="3.14159"/>
   <xacro:include filename="$(find taurob_erl_description)/urdf/taurob_chassis.urdf.xacro.xml" />
+<!--
   <xacro:include filename="$(find taurob_erl_description)/urdf/taurob_chassis_cameras.urdf.xacro.xml" />
   <xacro:tracker_chassis_cameras_macro />
+-->
   <!--LASER-->
-   <xacro:include filename="$(find taurob_erl_description)/urdf/hokuyo_utm30lx.urdf.xacro" />
+  <xacro:include filename="$(find taurob_erl_description)/urdf/hokuyo_utm30lx.urdf.xacro" />
   <!--schunk lwa4d arm-->
     <xacro:include filename="$(find taurob_schunk_lwa4d)/urdf/lwa4d/lwa4d.urdf.xacro" />
